File: LJ STAND/Main.sch (EAGLE design)
At the start: 210 parts, among them Q1 200mA/50V

Commit message: Light PCB routing
Parts:
- removed C14, C15: 22nF, SparkFun-Capacitors:CAP0805
- removed R43, R44: 1K, SparkFun-Resistors:RESISTOR0603-RES
Connections:
- removed net N$27: IR_1.OUT, R44.2
- removed net N$46: IR_0.OUT, R43.2
- net GND: no longer C14.2, C15.2
- net IR_0: now also IR_0.OUT; no longer C14.1, R43.1
- net IR_1: now also IR_1.OUT; no longer C15.1, R44.1
Changed lines of the file:
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@@
 <part name="SUPPLY17" library="SparkFun-Aesthetics" deviceset="3.3V" device=""/>
 <part name="GND20" library="SparkFun-Aesthetics" deviceset="GND" device=""/>
-<part name="R43" library="SparkFun-Resistors" deviceset="RESISTOR" device="0603-RES" value="1K"/>
-<part name="C14" library="SparkFun-Capacitors" deviceset="CAP" device="0805" value="22nF"/>
 <part name="IR_1" library="TSSP58038" deviceset="TSSP58038" device=""/>
 <part name="SUPPLY18" library="SparkFun-Aesthetics" deviceset="3.3V" device=""/>
 <part name="GND21" library="SparkFun-Aesthetics" deviceset="GND" device=""/>
-<part name="R44" library="SparkFun-Resistors" deviceset="RESISTOR" device="0603-RES" value="1K"/>
-<part name="C15" library="SparkFun-Capacitors" deviceset="CAP" device="0805" value="22nF"/>
 <part name="IR_2" library="TSSP58038" deviceset="TSSP58038" device=""/>
 <part name="SUPPLY19" library="SparkFun-Aesthetics" deviceset="3.3V" device=""/>
@@
 <instance part="IR_0" gate="G$1" x="177.8" y="-114.3" rot="R270"/>
 <instance part="SUPPLY17" gate="G$1" x="165.1" y="-104.14"/>
-<instance part="GND20" gate="1" x="157.48" y="-149.86"/>
-<instance part="R43" gate="G$1" x="165.1" y="-127" rot="R90"/>
-<instance part="C14" gate="G$1" x="165.1" y="-142.24"/>
+<instance part="GND20" gate="1" x="157.48" y="-119.38"/>
 <instance part="IR_1" gate="G$1" x="223.52" y="-114.3" rot="R270"/>
 <instance part="SUPPLY18" gate="G$1" x="210.82" y="-104.14"/>
-<instance part="GND21" gate="1" x="203.2" y="-149.86"/>
-<instance part="R44" gate="G$1" x="210.82" y="-127" rot="R90"/>
-<instance part="C15" gate="G$1" x="210.82" y="-142.24"/>
+<instance part="GND21" gate="1" x="203.2" y="-119.38"/>
 <instance part="IR_2" gate="G$1" x="266.7" y="-114.3" rot="R270"/>
 <instance part="SUPPLY19" gate="G$1" x="254" y="-104.14"/>
@@
 <pinref part="IR_0" gate="G$1" pin="GND"/>
 <wire x1="167.64" y1="-114.3" x2="157.48" y2="-114.3" width="0.1524" layer="91"/>
-<wire x1="157.48" y1="-114.3" x2="157.48" y2="-144.78" width="0.1524" layer="91"/>
+<wire x1="157.48" y1="-114.3" x2="157.48" y2="-116.84" width="0.1524" layer="91"/>
 <pinref part="GND20" gate="1" pin="GND"/>
-<pinref part="C14" gate="G$1" pin="2"/>
-<wire x1="157.48" y1="-144.78" x2="157.48" y2="-147.32" width="0.1524" layer="91"/>
-<wire x1="165.1" y1="-144.78" x2="157.48" y2="-144.78" width="0.1524" layer="91"/>
-<junction x="157.48" y="-144.78"/>
 <pinref part="C38" gate="G$1" pin="2"/>
 <junction x="157.48" y="-114.3"/>
@@
 <pinref part="IR_1" gate="G$1" pin="GND"/>
 <wire x1="213.36" y1="-114.3" x2="203.2" y2="-114.3" width="0.1524" layer="91"/>
-<wire x1="203.2" y1="-114.3" x2="203.2" y2="-144.78" width="0.1524" layer="91"/>
+<wire x1="203.2" y1="-114.3" x2="203.2" y2="-116.84" width="0.1524" layer="91"/>
 <pinref part="GND21" gate="1" pin="GND"/>
-<pinref part="C15" gate="G$1" pin="2"/>
-<wire x1="203.2" y1="-144.78" x2="203.2" y2="-147.32" width="0.1524" layer="91"/>
-<wire x1="210.82" y1="-144.78" x2="203.2" y2="-144.78" width="0.1524" layer="91"/>
-<junction x="203.2" y="-144.78"/>
 <pinref part="C39" gate="G$1" pin="2"/>
 <junction x="203.2" y="-114.3"/>
@@
 </segment>
 </net>
-<net name="IR_0" class="0">
-<segment>
-<pinref part="C14" gate="G$1" pin="1"/>
-<pinref part="R43" gate="G$1" pin="1"/>
-<wire x1="165.1" y1="-137.16" x2="165.1" y2="-134.62" width="0.1524" layer="91"/>
-<wire x1="165.1" y1="-134.62" x2="165.1" y2="-132.08" width="0.1524" layer="91"/>
-<wire x1="165.1" y1="-134.62" x2="170.18" y2="-134.62" width="0.1524" layer="91"/>
-<junction x="165.1" y="-134.62"/>
-<label x="170.18" y="-134.62" size="1.778" layer="95" xref="yes"/>
-</segment>
-<segment>
-<pinref part="SLAVE_SENSOR" gate="G$1" pin="0/RX1/MOSI1"/>
-<wire x1="205.74" y1="134.62" x2="203.2" y2="134.62" width="0.1524" layer="91"/>
-<label x="203.2" y="134.62" size="1.778" layer="95" rot="R180" xref="yes"/>
-</segment>
-</net>
-<net name="N$46" class="0">
-<segment>
-<pinref part="R43" gate="G$1" pin="2"/>
-<wire x1="165.1" y1="-121.92" x2="165.1" y2="-119.38" width="0.1524" layer="91"/>
-<pinref part="IR_0" gate="G$1" pin="OUT"/>
-<wire x1="165.1" y1="-119.38" x2="167.64" y2="-119.38" width="0.1524" layer="91"/>
-</segment>
-</net>
-<net name="N$27" class="0">
-<segment>
-<pinref part="R44" gate="G$1" pin="2"/>
-<wire x1="210.82" y1="-121.92" x2="210.82" y2="-119.38" width="0.1524" layer="91"/>
-<pinref part="IR_1" gate="G$1" pin="OUT"/>
-<wire x1="210.82" y1="-119.38" x2="213.36" y2="-119.38" width="0.1524" layer="91"/>
-</segment>
-</net>
 <net name="N$47" class="0">
 <segment>
@@
 <net name="IR_1" class="0">
 <segment>
-<pinref part="C15" gate="G$1" pin="1"/>
-<pinref part="R44" gate="G$1" pin="1"/>
-<wire x1="210.82" y1="-137.16" x2="210.82" y2="-134.62" width="0.1524" layer="91"/>
-<wire x1="210.82" y1="-134.62" x2="210.82" y2="-132.08" width="0.1524" layer="91"/>
-<wire x1="210.82" y1="-134.62" x2="215.9" y2="-134.62" width="0.1524" layer="91"/>
-<junction x="210.82" y="-134.62"/>
-<label x="215.9" y="-134.62" size="1.778" layer="95" xref="yes"/>
-</segment>
-<segment>
 <pinref part="SLAVE_SENSOR" gate="G$1" pin="1/TX1/MISO1"/>
 <wire x1="205.74" y1="129.54" x2="203.2" y2="129.54" width="0.1524" layer="91"/>
 <label x="203.2" y="129.54" size="1.778" layer="95" rot="R180" xref="yes"/>
 </segment>
+<segment>
+<wire x1="210.82" y1="-121.92" x2="210.82" y2="-119.38" width="0.1524" layer="91"/>
+<pinref part="IR_1" gate="G$1" pin="OUT"/>
+<wire x1="210.82" y1="-119.38" x2="213.36" y2="-119.38" width="0.1524" layer="91"/>
+<label x="210.82" y="-121.92" size="1.778" layer="95" rot="R270" xref="yes"/>
+</segment>
 </net>
 <net name="IR_2" class="0">
@@
 </segment>
 </net>
+<net name="IR_0" class="0">
+<segment>
+<pinref part="SLAVE_SENSOR" gate="G$1" pin="0/RX1/MOSI1"/>
+<wire x1="205.74" y1="134.62" x2="203.2" y2="134.62" width="0.1524" layer="91"/>
+<label x="203.2" y="134.62" size="1.778" layer="95" rot="R180" xref="yes"/>
+</segment>
+<segment>
+<pinref part="IR_0" gate="G$1" pin="OUT"/>
+<wire x1="165.1" y1="-119.38" x2="167.64" y2="-119.38" width="0.1524" layer="91"/>
+<label x="165.1" y="-121.92" size="1.778" layer="95" rot="R270" xref="yes"/>
+<wire x1="165.1" y1="-119.38" x2="165.1" y2="-121.92" width="0.1524" layer="91"/>
+</segment>
+</net>

Commit message: Finished routing light & encoder pcbs
Parts:
- removed C16, C17, C18, C19, C20, C21, C22, C23, C24, C25, C26, C27, C28, C29, C30, C31, C32, C33, C34, C35, C36, C37: 22nF, SparkFun-Capacitors:CAP0805
- removed R45, R46, R47, R48, R49, R50, R51, R52, R53, R54, R55, R56, R57, R58, R59, R60, R61, R62, R63, R64, R65, R66: 1K, SparkFun-Resistors:RESISTOR0603-RES
- added LS_CONNECTOR: (no value), pinhead+:PINHD-2X8SMT
- renumbered IR_0 to IR0, IR_1 to IR1, IR_10 to IR10, IR_11 to IR11, IR_12 to IR12, IR_13 to IR13, IR_14 to IR14, IR_15 to IR15, IR_16 to IR16, IR_17 to IR17, IR_18 to IR18, IR_19 to IR19, IR_2 to IR2, IR_20 to IR20, IR_21 to IR21, IR_22 to IR22, IR_23 to IR23, IR_3 to IR3, IR_4 to IR4, IR_5 to IR5, IR_6 to IR6, IR_7 to IR7, IR_8 to IR8, IR_9 to IR9
Connections:
- net IR_0 renamed IR0
- net IR_1 renamed IR1
- removed net IR_10: C24.1, R53.1, SLAVE_SENSOR.19/A5/SCL0
- removed net IR_11: C25.1, R54.1, SLAVE_SENSOR.20/A6/PWM/CS0
- removed net IR_12: C26.1, R55.1, SLAVE_SENSOR.21/A7/PWM/CS0
- removed net IR_13: C27.1, R56.1, SLAVE_SENSOR.22/A8/PWM
- removed net IR_14: C28.1, R57.1, SLAVE_SENSOR.23/A9/PWM
- removed net IR_15: C29.1, R58.1, SLAVE_SENSOR.24
- removed net IR_16: C30.1, R59.1, SLAVE_SENSOR.25
- removed net IR_17: C31.1, R60.1, SLAVE_SENSOR.26
- removed net IR_18: C32.1, R61.1, SLAVE_SENSOR.27
- removed net IR_19: C33.1, R62.1, SLAVE_SENSOR.28
- removed net IR_2: C16.1, R45.1, SLAVE_SENSOR.2/PWM
- removed net IR_20: C34.1, R63.1, SLAVE_SENSOR.29/PWM
- removed net IR_21: C35.1, R64.1, SLAVE_SENSOR.30/PWM
- removed net IR_22: C36.1, R65.1, SLAVE_SENSOR.31/A12/RX4/CS1
- removed net IR_23: C37.1, R66.1, SLAVE_SENSOR.32/A13/TX4/SCK1
- removed net IR_3: C17.1, R46.1, SLAVE_SENSOR.3/PWM/CAN0TX/SCL2
- removed net IR_4: C18.1, R47.1, SLAVE_SENSOR.4/PWM/CAN0RX/SDA2
- removed net IR_5: C19.1, R48.1, SLAVE_SENSOR.5/PWM
- removed net IR_6: C20.1, R49.1, SLAVE_SENSOR.6/PWM
- removed net IR_7: C21.1, R50.1, SLAVE_SENSOR.7/PWM/RX3
- removed net IR_8: C22.1, R51.1, SLAVE_SENSOR.8/PWM/TX3
- removed net IR_9: C23.1, R52.1, SLAVE_SENSOR.9/PWM/RX2/CS0
- removed net LS_0: SLAVE_SENSOR.14/A0/PWM
- removed net LS_1: SLAVE_SENSOR.15/A1/CS0
- removed net LS_2: SLAVE_SENSOR.16/A2
- removed net LS_3: SLAVE_SENSOR.17/A3
- removed net N$47: IR2.OUT, R45.2
- removed net N$48: IR3.OUT, R46.2
- removed net N$49: IR4.OUT, R47.2
- removed net N$50: IR5.OUT, R48.2
- removed net N$51: IR6.OUT, R49.2
- removed net N$52: IR7.OUT, R50.2
- removed net N$53: IR8.OUT, R51.2
- removed net N$54: IR9.OUT, R52.2
- removed net N$55: IR10.OUT, R53.2
- removed net N$56: IR11.OUT, R54.2
- removed net N$57: IR12.OUT, R55.2
- removed net N$58: IR13.OUT, R56.2
- removed net N$59: IR14.OUT, R57.2
- removed net N$60: IR15.OUT, R58.2
- removed net N$61: IR16.OUT, R59.2
- removed net N$62: IR17.OUT, R60.2
- removed net N$63: IR18.OUT, R61.2
- removed net N$64: IR19.OUT, R62.2
- removed net N$65: IR20.OUT, R63.2
- removed net N$66: IR21.OUT, R64.2
- removed net N$67: IR22.OUT, R65.2
- removed net N$68: IR23.OUT, R66.2
- new net IR10: IR10.OUT, SLAVE_SENSOR.19/A5/SCL0
- new net IR11: IR11.OUT, SLAVE_SENSOR.20/A6/PWM/CS0
- new net IR12: IR12.OUT, SLAVE_SENSOR.21/A7/PWM/CS0
- new net IR13: IR13.OUT, SLAVE_SENSOR.22/A8/PWM
- new net IR14: IR14.OUT, SLAVE_SENSOR.23/A9/PWM
- new net IR15: IR15.OUT, SLAVE_SENSOR.24
- new net IR16: IR16.OUT, SLAVE_SENSOR.25
- new net IR17: IR17.OUT, SLAVE_SENSOR.26
- new net IR18: IR18.OUT, SLAVE_SENSOR.27
- new net IR19: IR19.OUT, SLAVE_SENSOR.28
- new net IR2: IR2.OUT, SLAVE_SENSOR.2/PWM
- new net IR20: IR20.OUT, SLAVE_SENSOR.29/PWM
- new net IR21: IR21.OUT, SLAVE_SENSOR.30/PWM
- new net IR22: IR22.OUT, SLAVE_SENSOR.31/A12/RX4/CS1
- new net IR23: IR23.OUT, SLAVE_SENSOR.32/A13/TX4/SCK1
- new net IR3: IR3.OUT, SLAVE_SENSOR.3/PWM/CAN0TX/SCL2
- new net IR4: IR4.OUT, SLAVE_SENSOR.4/PWM/CAN0RX/SDA2
- new net IR5: IR5.OUT, SLAVE_SENSOR.5/PWM
- new net IR6: IR6.OUT, SLAVE_SENSOR.6/PWM
- new net IR7: IR7.OUT, SLAVE_SENSOR.7/PWM/RX3
- new net IR8: IR8.OUT, SLAVE_SENSOR.8/PWM/TX3
- new net IR9: IR9.OUT, SLAVE_SENSOR.9/PWM/RX2/CS0
- new net IR_PWR: C38.1, C39.1, C40.1, C41.1, C42.1, C43.1, C44.1, C45.1, C46.1, C47.1, C48.1, C49.1, C50.1, C51.1, C52.1, C53.1, C54.1, C55.1, C56.1, C57.1, C58.1, C59.1, C60.1, C61.1, IR0.VS, IR1.VS, IR10.VS, IR11.VS, IR12.VS, IR13.VS, IR14.VS, IR15.VS, IR16.VS, IR17.VS, IR18.VS, IR19.VS, IR2.VS, IR20.VS, IR21.VS, IR22.VS, IR23.VS, IR3.VS, IR4.VS, IR5.VS, IR6.VS, IR7.VS, IR8.VS, IR9.VS, SLAVE_SENSOR.43/CS2, SLAVE_SENSOR.44/MOSI2, SLAVE_SENSOR.45/MISO2
- new net LS0: LS_CONNECTOR.7, SLAVE_SENSOR.14/A0/PWM
- new net LS1: LS_CONNECTOR.5, SLAVE_SENSOR.15/A1/CS0
- new net LS2: LS_CONNECTOR.3, SLAVE_SENSOR.16/A2
- new net LS3: LS_CONNECTOR.1, SLAVE_SENSOR.17/A3
- new net MUX_A0: LS_CONNECTOR.4, SLAVE_SENSOR.33/A14/TX5
- new net MUX_A1: LS_CONNECTOR.2, SLAVE_SENSOR.34/A15/RX5
- new net MUX_A2: LS_CONNECTOR.6, SLAVE_SENSOR.35/A16/PWM
- new net MUX_A3: LS_CONNECTOR.8, SLAVE_SENSOR.36/A17/PWM
- new net MUX_A4: LS_CONNECTOR.10, SLAVE_SENSOR.37/A18/PWM/SCL1
- new net MUX_CS: LS_CONNECTOR.12, SLAVE_SENSOR.38/A19/PWM/SDA1
- new net MUX_EN: LS_CONNECTOR.16, SLAVE_SENSOR.46/SCK2
- new net MUX_WR: LS_CONNECTOR.14, SLAVE_SENSOR.39/A20
- net 3.3V: now also LS_CONNECTOR.9; no longer C38.1, C39.1, C40.1, C41.1, C42.1, C43.1, C44.1, C45.1, C46.1, C47.1, C48.1, C49.1, C50.1, C51.1, C52.1, C53.1, C54.1, C55.1, C56.1, C57.1, C58.1, C59.1, C60.1, C61.1, IR0.VS, IR1.VS, IR10.VS, IR11.VS, IR12.VS, IR13.VS, IR14.VS, IR15.VS, IR16.VS, IR17.VS, IR18.VS, IR19.VS, IR2.VS, IR20.VS, IR21.VS, IR22.VS, IR23.VS, IR3.VS, IR4.VS, IR5.VS, IR6.VS, IR7.VS, IR8.VS, IR9.VS
- net GND: now also LS_CONNECTOR.11, LS_CONNECTOR.13; no longer C16.2, C17.2, C18.2, C19.2, C20.2, C21.2, C22.2, C23.2, C24.2, C25.2, C26.2, C27.2, C28.2, C29.2, C30.2, C31.2, C32.2, C33.2, C34.2, C35.2, C36.2, C37.2
- net LS_MUX: now also LS_CONNECTOR.15

Commit message: Main PCB routing
Parts:
- added C14, C15, C16, C17: 0.1uF, SparkFun-Capacitors:CAP0805
- added LEDA1, LEDA2, LEDA3, LEDA4, LEDA5, LEDA6, LED_DEBUG1: RED, SparkFun-LED:LED0603
- added LEDD1, LEDD2, LEDD3, LEDD4, LEDD5, LEDD6, LED_DEBUG6: WHITE, SparkFun-LED:LED0603
- added LED_DEBUG2: GREEN, SparkFun-LED:LED0603
- added LED_DEBUG3: BLUE, SparkFun-LED:LED0603
- added LED_DEBUG4: ORANGE, SparkFun-LED:LED0603
- added LED_DEBUG5: YELLOW, SparkFun-LED:LED0603
- added LIGHT_GATE: (no value), jst-ph:B5B-PH-K-S
- added LOGIC_SWITCH, MOTOR_SWITCH: (no value), jst-vh:B2P-VH
- added Q2, Q3: (no value), SparkFun-DiscreteSemi:TRANSISTOR_NPNSOT23-3
- added R43, R44, R45, R46, R47, R48, R49, R50, R51, R52, R53, R54, R55, R56, R57, R58, R59, R60: 330, SparkFun-Resistors:RESISTOR0603-RES
- added R61, R62: 1K, SparkFun-Resistors:RESISTOR0603-RES
- added U$2: GYRO, Gyro:GYRO
- 3.3V_ON, 5V_ON: value (none) -> GREEN
- C2, C4, C5: value (none) -> 10uF
- C3: value (none) -> 22uF
Connections:
- removed net CAM_SCL: U$1.TXD/SCL
- removed net CAM_SDA: U$1.RXD/SDA
- new net CAM_RX: MASTER.7/PWM/RX3, U$1.TXD/SCL
- new net CAM_TX: MASTER.8/PWM/TX3, U$1.RXD/SDA
- new net GYRO_CS1: MASTER.43/CS2, U$2.CS1
- new net GYRO_CS2: MASTER.42, U$2.CS2
- new net GYRO_CS3: MASTER.54/CS2, U$2.CS3
- new net GYRO_MISO: MASTER.45/MISO2, U$2.MISO
- new net GYRO_MOSI: MASTER.44/MOSI2, U$2.MOSI
- new net GYRO_SCLK: MASTER.46/SCK2, U$2.SCLK
- new net LED_A_CTRL: R61.1, SLAVE_DEBUG.2/PWM
- new net LED_DEBUG1: R55.1, SLAVE_DEBUG.4/PWM/CAN0RX/SDA2
- new net LED_DEBUG2: R56.1, SLAVE_DEBUG.5/PWM
- new net LED_DEBUG3: R57.1, SLAVE_DEBUG.6/PWM
- new net LED_DEBUG4: R58.1, SLAVE_DEBUG.7/PWM/RX3
- new net LED_DEBUG5: R59.1, SLAVE_DEBUG.8/PWM/TX3
- new net LED_DEBUG6: R60.1, SLAVE_DEBUG.9/PWM/RX2/CS0
- new net LED_D_CTRL: R62.1, SLAVE_DEBUG.3/PWM/CAN0TX/SCL2
- new net LIGHT_GATE_LASER: LIGHT_GATE.3
- new net LIGHT_GATE_OUT: LIGHT_GATE.2
- new net N$1: MOTOR_FUSE.P1, MOTOR_SWITCH.2
- new net N$10: LEDA1.C, LEDA2.C, LEDA3.C, LEDA4.C, LEDA5.C, LEDA6.C, Q2.C
- new net N$2: LOGIC_FUSE.P1, LOGIC_SWITCH.1
- new net N$27: LEDD1.A, R49.2
- new net N$3: LEDA1.A, R43.2
- new net N$4: LEDA2.A, R44.2
- new net N$46: LEDD2.A, R50.2
- new net N$47: LEDD3.A, R51.2
- new net N$48: LEDD4.A, R52.2
- new net N$49: LEDD5.A, R53.2
- new net N$5: LEDA3.A, R45.2
- new net N$50: LEDD6.A, R54.2
- new net N$51: LEDD1.C, LEDD2.C, LEDD3.C, LEDD4.C, LEDD5.C, LEDD6.C, Q3.C
- new net N$52: LED_DEBUG1.A, R55.2
- new net N$53: LED_DEBUG2.A, R56.2
- new net N$54: LED_DEBUG3.A, R57.2
- new net N$55: LED_DEBUG4.A, R58.2
- new net N$56: LED_DEBUG5.A, R59.2
- new net N$57: LED_DEBUG6.A, R60.2
- new net N$58: Q2.B, R61.2
- new net N$59: Q3.B, R62.2
- new net N$6: LEDA4.A, R46.2
- new net N$61: LIGHT_GATE.4
- new net N$8: LEDA5.A, R47.2
- new net N$9: LEDA6.A, R48.2
- net 3.3V: now also C14.1, C15.1, C16.1, C17.1, LIGHT_GATE.1, MASTER.3.3V-1, R43.1, R44.1, R45.1, R46.1, R47.1, R48.1, R49.1, R50.1, R51.1, R52.1, R53.1, R54.1, SLAVE_DEBUG.3.3V-1, SLAVE_MOTOR.3.3V-1, SLAVE_SENSOR.3.3V-1, U$2.3.3V
- net GND: now also C14.2, C15.2, C16.2, C17.2, LED_DEBUG1.C, LED_DEBUG2.C, LED_DEBUG3.C, LED_DEBUG4.C, LED_DEBUG5.C, LED_DEBUG6.C, LIGHT_GATE.5, MASTER.AGND, MASTER.GND-1, MASTER.GND-2, MASTER.GND-3, MASTER.GND-4, Q2.E, Q3.E, SLAVE_DEBUG.AGND, SLAVE_DEBUG.GND, SLAVE_DEBUG.GND-1, SLAVE_DEBUG.GND-2, SLAVE_DEBUG.GND-3, SLAVE_DEBUG.GND-4, SLAVE_MOTOR.AGND, SLAVE_MOTOR.GND, SLAVE_MOTOR.GND-1, SLAVE_MOTOR.GND-2, SLAVE_MOTOR.GND-3, SLAVE_MOTOR.GND-4, SLAVE_SENSOR.AGND, SLAVE_SENSOR.GND, SLAVE_SENSOR.GND-1, SLAVE_SENSOR.GND-2, SLAVE_SENSOR.GND-3, SLAVE_SENSOR.GND-4, U$2.GND
- net N$12: now also LOGIC_SWITCH.2, MOTOR_SWITCH.1; no longer LOGIC_FUSE.P1, MOTOR_FUSE.P1
- net RGB_LED_DATA: now also SLAVE_DEBUG.23/A9/PWM
- net SCREEN_C/D: now also SLAVE_DEBUG.21/A7/PWM/CS0
- net SCREEN_CS: now also SLAVE_DEBUG.22/A8/PWM
- net SCREEN_D0: now also SLAVE_DEBUG.24
- net SCREEN_D1: now also SLAVE_DEBUG.25
- net SCREEN_D2: now also SLAVE_DEBUG.26
- net SCREEN_D3: now also SLAVE_DEBUG.27
- net SCREEN_D4: now also SLAVE_DEBUG.28
- net SCREEN_D5: now also SLAVE_DEBUG.29/PWM
- net SCREEN_D6: now also SLAVE_DEBUG.30/PWM
- net SCREEN_D7: now also SLAVE_DEBUG.31/A12/RX4/CS1
- net SCREEN_RD: now also SLAVE_DEBUG.19/A5/SCL0
- net SCREEN_WR: now also SLAVE_DEBUG.20/A6/PWM/CS0
- net SCREEN_X+: now also SLAVE_DEBUG.15/A1/CS0
- net SCREEN_X-: now also SLAVE_DEBUG.16/A2
- net SCREEN_Y+: now also SLAVE_DEBUG.17/A3
- net SCREEN_Y-: now also SLAVE_DEBUG.18/A4/SDA0
Other:
- moved on the sheet: C1, D1, PWR_IN, R1, R2

Commit message: Finished routing main pcb
Connections:
- removed net CAM_CS: U$1.SSEL
- removed net CAM_MISO: U$1.MISO
- removed net CAM_MOSI: U$1.MOSI
- removed net CAM_SCK: U$1.SCLK
Changed lines of the file:
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@@
-</segment>
-</net>
-<net name="CAM_CS" class="0">
-<segment>
-<pinref part="U$1" gate="G$1" pin="SSEL"/>
-<wire x1="-147.32" y1="83.82" x2="-144.78" y2="83.82" width="0.1524" layer="91"/>
-<label x="-144.78" y="83.82" size="1.778" layer="95" xref="yes"/>
-</segment>
-</net>
-<net name="CAM_SCK" class="0">
-<segment>
-<pinref part="U$1" gate="G$1" pin="SCLK"/>
-<wire x1="-147.32" y1="81.28" x2="-144.78" y2="81.28" width="0.1524" layer="91"/>
-<label x="-144.78" y="81.28" size="1.778" layer="95" xref="yes"/>
-</segment>
-</net>
-<net name="CAM_MISO" class="0">
-<segment>
-<pinref part="U$1" gate="G$1" pin="MISO"/>
-<wire x1="-147.32" y1="78.74" x2="-144.78" y2="78.74" width="0.1524" layer="91"/>
-<label x="-144.78" y="78.74" size="1.778" layer="95" xref="yes"/>
-</segment>
-</net>
-<net name="CAM_MOSI" class="0">
-<segment>
-<pinref part="U$1" gate="G$1" pin="MOSI"/>
-<wire x1="-147.32" y1="76.2" x2="-144.78" y2="76.2" width="0.1524" layer="91"/>
-<label x="-144.78" y="76.2" size="1.778" layer="95" xref="yes"/>
 </segment>
 </net>
@@
 </segment>
 <segment>
-<label x="444.5" y="101.6" size="1.778" layer="95" rot="R270" xref="yes"/>
+<label x="436.88" y="101.6" size="1.778" layer="95" rot="R90" xref="yes"/>
 <pinref part="R62" gate="G$1" pin="1"/>
-<wire x1="447.04" y1="101.6" x2="444.5" y2="101.6" width="0.1524" layer="91"/>
-</segment>
-</net>
+<wire x1="447.04" y1="101.6" x2="436.88" y2="101.6" width="0.1524" layer="91"/>
+</segment>
+</net>

Commit message: Some small fixes to the main pcb
Parts:
- R15, R24, R33, R42: value 1.5K -> 1K
Connections:
- net LIGHT_GATE_LASER: now also MASTER.21/A7/PWM/CS0, MASTER.22/A8/PWM, MASTER.23/A9/PWM
- net LIGHT_GATE_OUT: now also MASTER.20/A6/PWM/CS0
Changed lines of the file:
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@@
 <part name="SUPPLY9" library="SparkFun-Aesthetics" deviceset="3.3V" device=""/>
 <part name="R14" library="SparkFun-Resistors" deviceset="RESISTOR" device="0603-RES" value="10K"/>
-<part name="R15" library="SparkFun-Resistors" deviceset="RESISTOR" device="0603-RES" value="1.5K"/>
+<part name="R15" library="SparkFun-Resistors" deviceset="RESISTOR" device="0603-RES" value="1K"/>
 <part name="C6" library="SparkFun-Capacitors" deviceset="CAP" device="0805" value="33nF"/>
 <part name="GND11" library="SparkFun-Aesthetics" deviceset="GND" device=""/>
@@
 <part name="SUPPLY11" library="SparkFun-Aesthetics" deviceset="3.3V" device=""/>
 <part name="R23" library="SparkFun-Resistors" deviceset="RESISTOR" device="0603-RES" value="10K"/>
-<part name="R24" library="SparkFun-Resistors" deviceset="RESISTOR" device="0603-RES" value="1.5K"/>
+<part name="R24" library="SparkFun-Resistors" deviceset="RESISTOR" device="0603-RES" value="1K"/>
 <part name="C11" library="SparkFun-Capacitors" deviceset="CAP" device="0805" value="33nF"/>
 <part name="GND14" library="SparkFun-Aesthetics" deviceset="GND" device=""/>
@@
 <part name="SUPPLY13" library="SparkFun-Aesthetics" deviceset="3.3V" device=""/>
 <part name="R32" library="SparkFun-Resistors" deviceset="RESISTOR" device="0603-RES" value="10K"/>
-<part name="R33" library="SparkFun-Resistors" deviceset="RESISTOR" device="0603-RES" value="1.5K"/>
+<part name="R33" library="SparkFun-Resistors" deviceset="RESISTOR" device="0603-RES" value="1K"/>
 <part name="C12" library="SparkFun-Capacitors" deviceset="CAP" device="0805" value="33nF"/>
 <part name="GND16" library="SparkFun-Aesthetics" deviceset="GND" device=""/>
@@
 <part name="SUPPLY15" library="SparkFun-Aesthetics" deviceset="3.3V" device=""/>
 <part name="R41" library="SparkFun-Resistors" deviceset="RESISTOR" device="0603-RES" value="10K"/>
-<part name="R42" library="SparkFun-Resistors" deviceset="RESISTOR" device="0603-RES" value="1.5K"/>
+<part name="R42" library="SparkFun-Resistors" deviceset="RESISTOR" device="0603-RES" value="1K"/>
 <part name="C13" library="SparkFun-Capacitors" deviceset="CAP" device="0805" value="33nF"/>
 <part name="GND18" library="SparkFun-Aesthetics" deviceset="GND" device=""/>
@@
 </segment>
 </net>
-<net name="N$7" class="0">
-<segment>
-<wire x1="271.78" y1="116.84" x2="271.78" y2="119.38" width="0.1524" layer="91"/>
-</segment>
-</net>
 <net name="LED_A_CTRL" class="0">
 <segment>
@@
 <label x="-66.04" y="-2.54" size="1.778" layer="95" rot="R180" xref="yes"/>
 </segment>
+<segment>
+<pinref part="MASTER" gate="G$1" pin="20/A6/PWM/CS0"/>
+<wire x1="55.88" y1="109.22" x2="58.42" y2="109.22" width="0.1524" layer="91"/>
+<label x="58.42" y="109.22" size="1.778" layer="95" rot="R270" xref="yes"/>
+</segment>
 </net>
 <net name="LIGHT_GATE_LASER" class="0">
@@
 <label x="-66.04" y="-5.08" size="1.778" layer="95" rot="R180" xref="yes"/>
 </segment>
+<segment>
+<pinref part="MASTER" gate="G$1" pin="23/A9/PWM"/>
+<wire x1="55.88" y1="124.46" x2="58.42" y2="124.46" width="0.1524" layer="91"/>
+<pinref part="MASTER" gate="G$1" pin="21/A7/PWM/CS0"/>
+<wire x1="55.88" y1="114.3" x2="58.42" y2="114.3" width="0.1524" layer="91"/>
+<wire x1="58.42" y1="124.46" x2="58.42" y2="119.38" width="0.1524" layer="91"/>
+<wire x1="58.42" y1="119.38" x2="58.42" y2="114.3" width="0.1524" layer="91"/>
+<wire x1="58.42" y1="119.38" x2="73.66" y2="119.38" width="0.1524" layer="91"/>
+<pinref part="MASTER" gate="G$1" pin="22/A8/PWM"/>
+<wire x1="55.88" y1="119.38" x2="58.42" y2="119.38" width="0.1524" layer="91"/>
+<junction x="58.42" y="119.38"/>
+<label x="73.66" y="119.38" size="1.778" layer="95" rot="R270" xref="yes"/>
+</segment>
 </net>
