File: LJ STAND/Main.sch (EAGLE design)
At the start: 213 parts, among them Q1 200mA/50V

Commit message: Pin changes on teensys, removed some screen pins for motor grounding
Parts:
- C2, C4, C5: device SparkFun-Capacitors:CAP0603-CAP -> SparkFun-Capacitors:CAP0805
- C3: device SparkFun-Capacitors:CAP0603-CAP -> SparkFun-Capacitors:CAP1206
Connections:
- net GND: now also SCREEN.GND
- net GYRO_CS2: now also MASTER.55; no longer MASTER.42
- net IR_PWR: now also SLAVE_SENSOR.47/RX6, SLAVE_SENSOR.48/TX6, SLAVE_SENSOR.49/A23, SLAVE_SENSOR.50/A24
- net LS0: now also SLAVE_SENSOR.A22/DAC1; no longer SLAVE_SENSOR.14/A0/PWM
- net MOTOR1_CS: now also SLAVE_MOTOR.16/A2; no longer SLAVE_MOTOR.14/A0/PWM
- net MOTOR2_CS: now also SLAVE_MOTOR.17/A3; no longer SLAVE_MOTOR.15/A1/CS0
- net MOTOR3_CS: now also SLAVE_MOTOR.18/A4/SDA0; no longer SLAVE_MOTOR.16/A2
- net MOTOR4_CS: now also SLAVE_MOTOR.19/A5/SCL0; no longer SLAVE_MOTOR.17/A3
- net SCK: now also MASTER.14/A0/PWM, SLAVE_DEBUG.14/A0/PWM, SLAVE_MOTOR.14/A0/PWM, SLAVE_SENSOR.14/A0/PWM; no longer MASTER.13/SCK0, SLAVE_DEBUG.13/SCK0, SLAVE_MOTOR.13/SCK0, SLAVE_SENSOR.13/SCK0
- net V_BAT: now also SLAVE_DEBUG.A22/DAC1; no longer SLAVE_DEBUG.14/A0/PWM
Changed lines of the file:
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@@
 <part name="LOGIC_FUSE" library="fuse-holder-3568" deviceset="3568-FUSEHOLDER" device="" value="2A"/>
 <part name="VREG-3.3" library="linear" deviceset="LM340?-*" device="S" technology="05" value=""/>
-<part name="C2" library="SparkFun-Capacitors" deviceset="CAP" device="0603-CAP" value="10uF"/>
-<part name="C3" library="SparkFun-Capacitors" deviceset="CAP" device="0603-CAP" value="22uF"/>
-<part name="C4" library="SparkFun-Capacitors" deviceset="CAP" device="0603-CAP" value="10uF"/>
-<part name="C5" library="SparkFun-Capacitors" deviceset="CAP" device="0603-CAP" value="10uF"/>
+<part name="C2" library="SparkFun-Capacitors" deviceset="CAP" device="0805" value="10uF"/>
+<part name="C3" library="SparkFun-Capacitors" deviceset="CAP" device="1206" value="22uF"/>
+<part name="C4" library="SparkFun-Capacitors" deviceset="CAP" device="0805" value="10uF"/>
+<part name="C5" library="SparkFun-Capacitors" deviceset="CAP" device="0805" value="10uF"/>
 <part name="GND3" library="SparkFun-Aesthetics" deviceset="GND" device=""/>
 <part name="GND4" library="SparkFun-Aesthetics" deviceset="GND" device=""/>
@@
 <part name="GND100" library="SparkFun-Aesthetics" deviceset="GND" device=""/>
 <part name="GND101" library="SparkFun-Aesthetics" deviceset="GND" device=""/>
+<part name="GND102" library="SparkFun-Aesthetics" deviceset="GND" device=""/>
 </parts>
 <sheets>
@@
 <instance part="GND85" gate="1" x="99.06" y="134.62"/>
 <instance part="GND86" gate="1" x="193.04" y="134.62"/>
-<instance part="GND87" gate="1" x="269.24" y="63.5"/>
+<instance part="GND87" gate="1" x="279.4" y="66.04"/>
 <instance part="GND88" gate="1" x="185.42" y="12.7"/>
 <instance part="GND89" gate="1" x="203.2" y="-43.18"/>
 <instance part="GND90" gate="1" x="236.22" y="-73.66"/>
 <instance part="GND91" gate="1" x="302.26" y="134.62"/>
-<instance part="GND92" gate="1" x="368.3" y="63.5"/>
+<instance part="GND92" gate="1" x="383.54" y="66.04"/>
 <instance part="GND93" gate="1" x="302.26" y="12.7"/>
 <instance part="GND94" gate="1" x="302.26" y="-43.18"/>
@@
 <instance part="GND100" gate="1" x="-132.08" y="-33.02"/>
 <instance part="GND101" gate="1" x="-132.08" y="-99.06"/>
+<instance part="GND102" gate="1" x="-248.92" y="-139.7"/>
 </instances>
 <busses>
@@
 <net name="SCK" class="0">
 <segment>
-<pinref part="SLAVE_DEBUG" gate="G$1" pin="13/SCK0"/>
-<wire x1="365.76" y1="73.66" x2="368.3" y2="73.66" width="0.1524" layer="91"/>
-<label x="368.3" y="73.66" size="1.778" layer="95" xref="yes"/>
+<pinref part="MASTER" gate="G$1" pin="14/A0/PWM"/>
+<wire x1="55.88" y1="78.74" x2="58.42" y2="78.74" width="0.1524" layer="91"/>
+<label x="58.42" y="78.74" size="1.778" layer="95" xref="yes"/>
 </segment>
 <segment>
-<pinref part="SLAVE_SENSOR" gate="G$1" pin="13/SCK0"/>
-<wire x1="266.7" y1="73.66" x2="269.24" y2="73.66" width="0.1524" layer="91"/>
-<label x="269.24" y="73.66" size="1.778" layer="95" xref="yes"/>
+<pinref part="SLAVE_MOTOR" gate="G$1" pin="14/A0/PWM"/>
+<wire x1="162.56" y1="78.74" x2="165.1" y2="78.74" width="0.1524" layer="91"/>
+<label x="165.1" y="78.74" size="1.778" layer="95" xref="yes"/>
 </segment>
 <segment>
-<pinref part="SLAVE_MOTOR" gate="G$1" pin="13/SCK0"/>
-<wire x1="162.56" y1="73.66" x2="165.1" y2="73.66" width="0.1524" layer="91"/>
-<label x="165.1" y="73.66" size="1.778" layer="95" xref="yes"/>
+<pinref part="SLAVE_DEBUG" gate="G$1" pin="14/A0/PWM"/>
+<wire x1="365.76" y1="78.74" x2="368.3" y2="78.74" width="0.1524" layer="91"/>
+<label x="368.3" y="78.74" size="1.778" layer="95" xref="yes"/>
 </segment>
 <segment>
-<pinref part="MASTER" gate="G$1" pin="13/SCK0"/>
-<wire x1="55.88" y1="73.66" x2="58.42" y2="73.66" width="0.1524" layer="91"/>
-<label x="58.42" y="73.66" size="1.778" layer="95" xref="yes"/>
+<pinref part="SLAVE_SENSOR" gate="G$1" pin="14/A0/PWM"/>
+<wire x1="266.7" y1="78.74" x2="269.24" y2="78.74" width="0.1524" layer="91"/>
+<label x="269.24" y="78.74" size="1.778" layer="95" xref="yes"/>
 </segment>
 </net>
@@
 </segment>
 <segment>
-<pinref part="SLAVE_DEBUG" gate="G$1" pin="14/A0/PWM"/>
-<wire x1="365.76" y1="78.74" x2="368.3" y2="78.74" width="0.1524" layer="91"/>
-<label x="368.3" y="78.74" size="1.778" layer="95" xref="yes"/>
+<pinref part="SLAVE_DEBUG" gate="G$1" pin="A22/DAC1"/>
+<wire x1="365.76" y1="63.5" x2="368.3" y2="63.5" width="0.1524" layer="91"/>
+<label x="368.3" y="63.5" size="1.778" layer="95" xref="yes"/>
 </segment>
 </net>
@@
 <segment>
 <pinref part="SLAVE_SENSOR" gate="G$1" pin="GND-1"/>
-<wire x1="266.7" y1="68.58" x2="269.24" y2="68.58" width="0.1524" layer="91"/>
-<wire x1="269.24" y1="68.58" x2="269.24" y2="66.04" width="0.1524" layer="91"/>
+<wire x1="266.7" y1="68.58" x2="279.4" y2="68.58" width="0.1524" layer="91"/>
 <pinref part="GND87" gate="1" pin="GND"/>
 </segment>
@@
 <segment>
 <pinref part="SLAVE_DEBUG" gate="G$1" pin="GND-1"/>
-<wire x1="365.76" y1="68.58" x2="368.3" y2="68.58" width="0.1524" layer="91"/>
-<wire x1="368.3" y1="68.58" x2="368.3" y2="66.04" width="0.1524" layer="91"/>
+<wire x1="365.76" y1="68.58" x2="383.54" y2="68.58" width="0.1524" layer="91"/>
 <pinref part="GND92" gate="1" pin="GND"/>
 </segment>
@@
 <wire x1="-132.08" y1="-27.94" x2="-132.08" y2="-30.48" width="0.1524" layer="91"/>
 </segment>
+<segment>
+<pinref part="SCREEN" gate="G$1" pin="GND"/>
+<wire x1="-243.84" y1="-134.62" x2="-248.92" y2="-134.62" width="0.1524" layer="91"/>
+<wire x1="-248.92" y1="-134.62" x2="-248.92" y2="-137.16" width="0.1524" layer="91"/>
+<pinref part="GND102" gate="1" pin="GND"/>
+</segment>
 </net>
 <net name="N$12" class="0">
@@
 </segment>
 <segment>
-<pinref part="SLAVE_MOTOR" gate="G$1" pin="17/A3"/>
-<wire x1="162.56" y1="93.98" x2="165.1" y2="93.98" width="0.1524" layer="91"/>
-<label x="165.1" y="93.98" size="1.778" layer="95" xref="yes"/>
+<pinref part="SLAVE_MOTOR" gate="G$1" pin="19/A5/SCL0"/>
+<wire x1="162.56" y1="104.14" x2="165.1" y2="104.14" width="0.1524" layer="91"/>
+<label x="165.1" y="104.14" size="1.778" layer="95" xref="yes"/>
 </segment>
 </net>
@@
 </segment>
 <segment>
-<pinref part="SLAVE_MOTOR" gate="G$1" pin="14/A0/PWM"/>
-<wire x1="162.56" y1="78.74" x2="165.1" y2="78.74" width="0.1524" layer="91"/>
-<label x="165.1" y="78.74" size="1.778" layer="95" xref="yes"/>
+<pinref part="SLAVE_MOTOR" gate="G$1" pin="16/A2"/>
+<wire x1="162.56" y1="88.9" x2="165.1" y2="88.9" width="0.1524" layer="91"/>
+<label x="165.1" y="88.9" size="1.778" layer="95" xref="yes"/>
 </segment>
 </net>
@@
 </segment>
 <segment>
-<pinref part="SLAVE_MOTOR" gate="G$1" pin="15/A1/CS0"/>
-<wire x1="162.56" y1="83.82" x2="165.1" y2="83.82" width="0.1524" layer="91"/>
-<label x="165.1" y="83.82" size="1.778" layer="95" xref="yes"/>
+<pinref part="SLAVE_MOTOR" gate="G$1" pin="17/A3"/>
+<wire x1="162.56" y1="93.98" x2="165.1" y2="93.98" width="0.1524" layer="91"/>
+<label x="165.1" y="93.98" size="1.778" layer="95" xref="yes"/>
 </segment>
 </net>
@@
 </segment>
 <segment>
-<pinref part="SLAVE_MOTOR" gate="G$1" pin="16/A2"/>
-<wire x1="162.56" y1="88.9" x2="165.1" y2="88.9" width="0.1524" layer="91"/>
-<label x="165.1" y="88.9" size="1.778" layer="95" xref="yes"/>
+<pinref part="SLAVE_MOTOR" gate="G$1" pin="18/A4/SDA0"/>
+<wire x1="162.56" y1="99.06" x2="165.1" y2="99.06" width="0.1524" layer="91"/>
+<label x="165.1" y="99.06" size="1.778" layer="95" xref="yes"/>
 </segment>
 </net>
@@
 <net name="LS0" class="0">
 <segment>
-<pinref part="SLAVE_SENSOR" gate="G$1" pin="14/A0/PWM"/>
-<wire x1="266.7" y1="78.74" x2="269.24" y2="78.74" width="0.1524" layer="91"/>
-<label x="269.24" y="78.74" size="1.778" layer="95" xref="yes"/>
-</segment>
-<segment>
 <pinref part="LS_CONNECTOR" gate="A" pin="7"/>
 <wire x1="-76.2" y1="66.04" x2="-81.28" y2="66.04" width="0.1524" layer="91"/>
 <label x="-81.28" y="66.04" size="1.778" layer="95" rot="R180" xref="yes"/>
 </segment>
+<segment>
+<pinref part="SLAVE_SENSOR" gate="G$1" pin="A22/DAC1"/>
+<wire x1="266.7" y1="63.5" x2="269.24" y2="63.5" width="0.1524" layer="91"/>
+<label x="269.24" y="63.5" size="1.778" layer="95" xref="yes"/>
+</segment>
 </net>
 <net name="LS1" class="0">
@@
 <label x="200.66" y="2.54" size="1.778" layer="95" rot="R180" xref="yes"/>
 </segment>
+<segment>
+<pinref part="SLAVE_SENSOR" gate="G$1" pin="48/TX6"/>
+<wire x1="266.7" y1="7.62" x2="269.24" y2="7.62" width="0.1524" layer="91"/>
+<wire x1="269.24" y1="7.62" x2="269.24" y2="2.54" width="0.1524" layer="91"/>
+<pinref part="SLAVE_SENSOR" gate="G$1" pin="49/A23"/>
+<wire x1="269.24" y1="2.54" x2="266.7" y2="2.54" width="0.1524" layer="91"/>
+<pinref part="SLAVE_SENSOR" gate="G$1" pin="50/A24"/>
+<wire x1="266.7" y1="-2.54" x2="269.24" y2="-2.54" width="0.1524" layer="91"/>
+<wire x1="269.24" y1="-2.54" x2="269.24" y2="2.54" width="0.1524" layer="91"/>
+<wire x1="269.24" y1="2.54" x2="271.78" y2="2.54" width="0.1524" layer="91"/>
+<junction x="269.24" y="2.54"/>
+<label x="271.78" y="2.54" size="1.778" layer="95" xref="yes"/>
+<pinref part="SLAVE_SENSOR" gate="G$1" pin="47/RX6"/>
+<wire x1="266.7" y1="12.7" x2="269.24" y2="12.7" width="0.1524" layer="91"/>
+<wire x1="269.24" y1="12.7" x2="269.24" y2="7.62" width="0.1524" layer="91"/>
+<junction x="269.24" y="7.62"/>
+</segment>
 </net>
 <net name="N$1" class="0">
@@
 </segment>
 <segment>
-<pinref part="MASTER" gate="G$1" pin="42"/>
-<wire x1="-5.08" y1="-7.62" x2="-7.62" y2="-7.62" width="0.1524" layer="91"/>
-<label x="-7.62" y="-7.62" size="1.778" layer="95" rot="R180" xref="yes"/>
+<pinref part="MASTER" gate="G$1" pin="55"/>
+<wire x1="55.88" y1="-27.94" x2="58.42" y2="-27.94" width="0.1524" layer="91"/>
+<label x="58.42" y="-27.94" size="1.778" layer="95" xref="yes"/>
 </segment>
 </net>
